Commit message: Added simulated camera mux

File: ros_workspace/src/rov_description/urdf/rov_sensors.xacro (robot description, xacro)
@@ -83,5 +83,5 @@
           <imageTopicName>image_raw</imageTopicName>
           <cameraInfoTopicName>camera_info</cameraInfoTopicName>
-          <frameName>camera_link</frameName>
+          <frameName>camera${number}_link</frameName>
           <hackBaseline>0.07</hackBaseline>
           <distortionK1>0.0</distortionK1>
@@ -101,8 +101,8 @@
   </xacro:camera_macro>
   <xacro:camera_macro number="2" parent="${namespace}/frame_link">
-    <origin xyz="0.05 0 -0.05" rpy="0 0 ${0*d2r}"/>
+    <origin xyz="0.05 0 -0.04" rpy="0 0 ${0*d2r}"/>
   </xacro:camera_macro>
   <xacro:camera_macro number="4" parent="${namespace}/frame_link">
-    <origin xyz="-0.05 0 -0.05" rpy="0 0 ${180*d2r}"/>
+    <origin xyz="-0.05 0 -0.04" rpy="0 0 ${180*d2r}"/>
   </xacro:camera_macro>
 </robot>
