Commit message: Updated meshes coordinate system and added proper collision geometry

File: ros_workspace/src/rov_description/urdf/rov.gazebo.xacro (robot description, xacro)
@@ -1,5 +1,5 @@
 <?xml version="1.0"?>
 <robot xmlns:xacro="http://www.ros.org/wiki/xacro">
-    <xacro:property name="cob" value="-0.00037196 -0.05465685 0.03359269"/>
+    <xacro:property name="cob" value="0.00037196 0.03359269 -0.05465685"/>
     <xacro:property name="volume" value="0.00980413"/>
     <xacro:macro name="rov_hydro_model" params="namespace">

File: ros_workspace/src/rov_description/urdf/rov_actuators.xacro (robot description, xacro)
@@ -1,5 +1,4 @@
 <?xml version="1.0"?>
 <robot xmlns:xacro="http://www.ros.org/wiki/xacro">
-  <!-- <xacro:property name="prop_mesh_file" value="file://$(find rov_description)/meshes/T100_cw_propeller.STL"/> -->
   <!-- Thruster joint and link snippet -->
   <xacro:macro name="thruster_macro"

File: ros_workspace/src/rov_description/urdf/rov_base.xacro (robot description, xacro)
@@ -6,7 +6,10 @@
   <xacro:include filename="$(find uuv_gazebo_ros_plugins)/urdf/snippets.xacro"/>
   <!-- Parameters -->
-  <xacro:property name="namespace" value="sim"/>
+  <xacro:property name="namespace" value="rov"/>
   <xacro:property name="visual_mesh_file" value="file://$(find rov_description)/meshes/rov_frame.STL"/>
   <xacro:property name="prop_mesh_file" value="file://$(find rov_description)/meshes/T100_cw_propeller.STL"/>
+  <!-- Constants -->
+  <xacro:property name="deg2rad" value="0.0174532925"/>
+  <xacro:property name="deg90" value="1.570796327"/>
   <!-- Mass -->
   <xacro:property name="mass" value="9.80543312"/>
@@ -16,8 +19,8 @@
       <inertial>
         <mass value="${mass}"/>
-        <origin xyz="-0.00056715 -0.12001042 0.01957420"/> <!-- center of mass -->
-        <inertia ixx = "0.24968270"  ixy = "0.00076418"  ixz = "-0.00003120"
-                 iyx = "0.00076418"  iyy = "0.22666109"  iyz = "-0.01991623"
-                 izx = "-0.00003120" izy = "-0.01991623" izz = "0.19606323"/>
+        <origin xyz="0.00056715 0.01957420 -0.12001042"/> <!-- center of mass -->
+        <inertia ixx = "0.24968270"  ixy = "0.00003120"  ixz = "-0.00076418"
+                 iyx = "0.00003120"  iyy = "0.19606323"  iyz = "-0.01991623"
+                 izx = "-0.00076418" izy = "-0.01991623" izz = "0.22666109" />
       </inertial>
       <visual>
@@ -29,5 +32,5 @@
       <!-- bottom frame -->
       <collision>
-        <origin xyz="0 0 -0.264" rpy="0 0 0"/>
+        <origin xyz="0 0.0373 -0.25" rpy="0 0 ${deg90}"/>
         <geometry>
           <box size="0.375 0.220 -0.015"/>
@@ -36,25 +39,25 @@
       <!-- top frame -->
       <collision>
-        <origin xyz="0 0 -0.05" rpy="0 0 0"/>
-        <geometry><box size="0.32279107 0.39804338 0.05856"/></geometry>
+        <origin xyz="0 0.0373 -0.05" rpy="${deg90} 0 0"/>
+        <geometry><box size="0.32279107 0.05856 0.39804338"/></geometry>
       </collision>
       <!-- left front leg -->
       <collision>
-        <origin xyz="0.23 0.105 -0.193" rpy="0 0 0"/>
+        <origin xyz="0.1 0.21 -0.16" rpy="0 ${deg90} 0"/>
         <geometry><box size="0.178 0.02 0.02"/></geometry>
       </collision>
       <!-- right front leg -->
       <collision>
-        <origin xyz="0.23 -0.105 -0.193" rpy="0 0 0"/>
+        <origin xyz="-0.1 0.21 -0.16" rpy="0 ${deg90} 0"/>
         <geometry><box size="0.178 0.02 0.02"/></geometry>
       </collision>
       <!-- left back leg -->
       <collision>
-        <origin xyz="-0.15265 0.105 -0.193" rpy="0 0 0"/>
+        <origin xyz="0.1 -0.135 -0.16" rpy="0 ${deg90} 0"/>
         <geometry><box size="0.178 0.02 0.02"/></geometry>
       </collision>
       <!-- right back leg -->
       <collision>
-        <origin xyz="-0.15265 -0.105 -0.193" rpy="0 0 0"/>
+        <origin xyz="-0.1 -0.135 -0.16" rpy="0 ${deg90} 0"/>
         <geometry><box size="0.178 0.02 0.02"/></geometry>
       </collision>

File: ros_workspace/src/rov_description/urdf/rov_default.xacro (robot description, xacro)
@@ -11,5 +11,5 @@
     <parent link="${namespace}/base_link"/>
     <child link="${namespace}/frame_link"/>
-    <origin xyz="0 0.15585 -0.0373" rpy="0 0 0"/>
+    <origin xyz="0 -0.0373 0.15585" rpy="0 0 0"/>
   </joint>
   <!-- Create the rov sim model -->
@@ -30,4 +30,4 @@
   </xacro:rov_base>
   <!-- Joint state publisher plugin -->
-  <xacro:default_joint_state_publisher namespace="$(arg namespace)" update_rate="50"/>
+  <!--<xacro:default_joint_state_publisher namespace="$(arg namespace)" update_rate="50"/>-->
 </robot>

Commit message: base working model

File: ros_workspace/src/rov_description/urdf/rov.gazebo.xacro (robot description, xacro)
@@ -4,16 +4,16 @@
     <xacro:property name="volume" value="0.00980413"/>
     <xacro:macro name="rov_hydro_model" params="namespace">
-        <link name="${namespace}/frame_link">
+        <link name="${namespace}/base_link">
             <neutrally_buoyant>0</neutrally_buoyant>
             <volume>${volume}</volume>
             <box>
-                <width>0.61075</width>
-                <length>0.030617</length>
-                <height>0.46237</height>
+              <width>0.61075</width>
+              <length>0.030617</length>
+              <height>0.46237</height>
             </box>
             <center_of_buoyancy>${cob}</center_of_buoyancy>
             <hydrodynamic_model>
               <type>sphere</type>
-              <radius>0.305375</radius>
+              <radius>0.3</radius>
             </hydrodynamic_model>
         </link>

File: ros_workspace/src/rov_description/urdf/rov_base.xacro (robot description, xacro)
@@ -16,5 +16,5 @@
   <xacro:macro name="rov_base" params="namespace *gazebo inertial_reference_frame">
     <!-- base_link according to ROS conventions: x forward, z up -->
-    <link name="${namespace}/frame_link">
+    <link name="${namespace}/base_link">
       <inertial>
         <mass value="${mass}"/>
@@ -72,5 +72,5 @@
     </gazebo> -->
     <xacro:include filename="$(find rov_description)/urdf/rov_actuators.xacro"/>
-    <xacro:include filename="$(find rov_description)/urdf/rov_sensors.xacro"/>
+    <!-- <xacro:include filename="$(find rov_description)/urdf/rov_sensors.xacro"/> -->
   </xacro:macro>
 </robot>

File: ros_workspace/src/rov_description/urdf/rov_default.xacro (robot description, xacro)
@@ -1,4 +1,5 @@
 <?xml version="1.0"?>
 <robot name="rov" xmlns:xacro="http://www.ros.org/wiki/xacro" >
+  <xacro:arg name="debug" default="0"/>
   <xacro:arg name="namespace" default="rov"/>
   <xacro:arg name="inertial_reference_frame" default="world"/>
@@ -7,11 +8,11 @@
   <xacro:include filename="$(find rov_description)/urdf/rov.gazebo.xacro"/>
   <!-- setup base links -->
-  <link name="${namespace}/base_link"/>
+  <link name="${namespace}/frame_link"/>
   <joint name="base_link_joint" type="fixed">
-    <parent link="${namespace}/base_link"/>
-    <child link="${namespace}/frame_link"/>
+    <parent link="${namespace}/frame_link"/>
+    <child link="${namespace}/base_link"/>
     <origin xyz="0 -0.0373 0.15585" rpy="0 0 0"/>
   </joint>
-  <!-- Create the rov sim model -->
+  <!-- Create the rov -->
   <xacro:rov_base
     namespace="$(arg namespace)"
@@ -21,7 +22,7 @@
     <gazebo>
       <plugin name="uuv_plugin" filename="libuuv_underwater_object_ros_plugin.so">
-        <fluid_density>1028.0</fluid_density>
+        <fluid_density>1000.0</fluid_density>
         <flow_velocity_topic>hydrodynamics/current_velocity</flow_velocity_topic>
-        <debug>0</debug>
+        <debug>$(arg debug)</debug>
         <!-- Adding the hydrodynamic and hydrostatic parameters for the vehicle-->
         <xacro:rov_hydro_model namespace="$(arg namespace)"/>
@@ -30,4 +31,4 @@
   </xacro:rov_base>
   <!-- Joint state publisher plugin -->
-  <!--<xacro:default_joint_state_publisher namespace="$(arg namespace)" update_rate="50"/>-->
+  <xacro:default_joint_state_publisher namespace="$(arg namespace)" update_rate="50"/>
 </robot>

Commit message: Smaller more optimized mesh

File: ros_workspace/src/rov_description/urdf/rov.gazebo.xacro (robot description, xacro)
@@ -1,6 +1,6 @@
 <?xml version="1.0"?>
 <robot xmlns:xacro="http://www.ros.org/wiki/xacro">
-    <xacro:property name="cob" value="0.00037196 0.03359269 -0.05465685"/>
-    <xacro:property name="volume" value="0.00980413"/>
+    <xacro:property name="cob" value="0.0 0.0 -0.05465685"/>
+    <xacro:property name="volume" value="0.01"/>
     <xacro:macro name="rov_hydro_model" params="namespace">
         <link name="${namespace}/base_link">
@@ -16,4 +16,22 @@
               <type>sphere</type>
               <radius>0.3</radius>
+              <!-- <type>fossen</type> -->
+              <!-- Added mass: see p.28 in Berg2012 -->
+              <!-- <added_mass>
+                   779.79 -6.8773 -103.32  8.5426 -165.54 -7.8033
+                  -6.8773    1222   51.29  409.44 -5.8488  62.726
+                  -103.32   51.29  3659.9  6.1112 -386.42  10.774
+                   8.5426  409.44  6.1112   534.9 -10.027  21.019
+                  -165.54 -5.8488 -386.42 -10.027  842.69 -1.1162
+                  -7.8033  62.726  10.775  21.019 -1.1162  224.32
+              </added_mass> -->
+              <!-- Linear damping: see p.31 in Berg2012 -->
+              <!-- <linear_damping>
+                  -74.82 -69.48 -728.4 -268.8 -309.77 -105
+              </linear_damping> -->
+              <!-- Non-linear damping: see p.30 in Berg2012 -->
+              <!-- <quadratic_damping>
+                  -748.22 -992.53 -1821.01 -672 -774.44 -523.27
+              </quadratic_damping> -->
             </hydrodynamic_model>
         </link>

File: ros_workspace/src/rov_description/urdf/rov_base.xacro (robot description, xacro)
@@ -19,5 +19,5 @@
       <inertial>
         <mass value="${mass}"/>
-        <origin xyz="0.00056715 0.01957420 -0.12001042"/> <!-- center of mass -->
+        <origin xyz="0.0 0.0 -0.12001042"/> <!-- center of mass -->
         <inertia ixx = "0.24968270"  ixy = "0.00003120"  ixz = "-0.00076418"
                  iyx = "0.00003120"  iyy = "0.19606323"  iyz = "-0.01991623"

File: ros_workspace/src/rov_description/urdf/rov_default.xacro (robot description, xacro)
@@ -7,11 +7,4 @@
   <xacro:include filename="$(find rov_description)/urdf/rov_base.xacro"/>
   <xacro:include filename="$(find rov_description)/urdf/rov.gazebo.xacro"/>
-  <!-- setup base links -->
-  <link name="${namespace}/frame_link"/>
-  <joint name="base_link_joint" type="fixed">
-    <parent link="${namespace}/frame_link"/>
-    <child link="${namespace}/base_link"/>
-    <origin xyz="0 -0.0373 0.15585" rpy="0 0 0"/>
-  </joint>
   <!-- Create the rov -->
   <xacro:rov_base
@@ -30,4 +23,11 @@
     </gazebo>
   </xacro:rov_base>
+  <!-- setup base links -->
+  <link name="${namespace}/frame_link"/>
+  <joint name="base_link_joint" type="fixed">
+    <parent link="${namespace}/base_link"/>
+    <child link="${namespace}/frame_link"/>
+    <origin xyz="0 0.0373 -0.15585" rpy="0 0 0"/>
+  </joint>
   <!-- Joint state publisher plugin -->
   <xacro:default_joint_state_publisher namespace="$(arg namespace)" update_rate="50"/>

Commit message: rough thruster arrangement

File: ros_workspace/src/rov_description/urdf/rov.gazebo.xacro (robot description, xacro)
@@ -15,5 +15,5 @@
             <hydrodynamic_model>
               <type>sphere</type>
-              <radius>0.3</radius>
+              <radius>1</radius>
               <!-- <type>fossen</type> -->
               <!-- Added mass: see p.28 in Berg2012 -->

File: ros_workspace/src/rov_description/urdf/rov_actuators.xacro (robot description, xacro)
@@ -14,20 +14,20 @@
   </xacro:macro>
   <xacro:thruster_macro namespace="${namespace}" thruster_id="1">
-    <origin xyz="0.230 0.1587 -0.13603" rpy="${0*d2r} ${-74.53*d2r} ${-53.21*d2r}"/>
+    <origin xyz="-0.1587 0.228 -0.14" rpy="${90*d2r} ${0*d2r} ${-225*d2r}"/>
   </xacro:thruster_macro>
   <xacro:thruster_macro namespace="${namespace}" thruster_id="2">
-    <origin xyz="0.230 -0.1587 -0.13603" rpy="${0*d2r} ${-74.53*d2r} ${53.21*d2r}"/>
+    <origin xyz="0.1587 0.228 -0.14" rpy="${90*d2r} ${0*d2r} ${225*d2r}"/>
   </xacro:thruster_macro>
   <xacro:thruster_macro namespace="${namespace}" thruster_id="3">
-    <origin xyz="-0.15265 -0.1587 -0.13603" rpy="${0*d2r} ${-105.47*d2r} ${53.21*d2r}"/>
+    <origin xyz="0.16 -0.157 -0.132" rpy="${90*d2r} ${0*d2r} ${-45*d2r}"/>
   </xacro:thruster_macro>
   <xacro:thruster_macro namespace="${namespace}" thruster_id="4">
-    <origin xyz="-0.15265 0.1587 -0.13603" rpy="${0*d2r} ${-105.47*d2r} ${-53.21*d2r}"/>
+    <origin xyz="-0.16 -0.157 -0.132" rpy="${90*d2r} ${0*d2r} ${45*d2r}"/>
   </xacro:thruster_macro>
   <xacro:thruster_macro namespace="${namespace}" thruster_id="5">
-    <origin xyz="0.03394 0.25550 -0.8263" rpy="${0*d2r} ${0*d2r} ${45*d2r}"/>
+    <origin xyz="-0.25550 0.03394 -0.08263" rpy="${0*d2r} ${0*d2r} ${0*d2r}"/>
   </xacro:thruster_macro>
   <xacro:thruster_macro namespace="${namespace}" thruster_id="6">
-    <origin xyz="0.03394 -0.25550 -0.8263" rpy="${0*d2r} ${0*d2r} ${-45*d2r}"/>
+    <origin xyz="0.25550 0.03394 -0.08263" rpy="${0*d2r} ${0*d2r} ${0*d2r}"/>
   </xacro:thruster_macro>
 </robot>

Commit message: Working Simulation model

File: ros_workspace/src/rov_description/urdf/rov.gazebo.xacro (robot description, xacro)
@@ -1,5 +1,5 @@
 <?xml version="1.0"?>
 <robot xmlns:xacro="http://www.ros.org/wiki/xacro">
-    <xacro:property name="cob" value="0.0 0.0 -0.05465685"/>
+    <xacro:property name="cob" value="0.0 0.0 0.01"/>
     <xacro:property name="volume" value="0.01"/>
     <xacro:macro name="rov_hydro_model" params="namespace">
@@ -14,9 +14,9 @@
             <center_of_buoyancy>${cob}</center_of_buoyancy>
             <hydrodynamic_model>
-              <type>sphere</type>
-              <radius>1</radius>
-              <!-- <type>fossen</type> -->
+              <!-- <type>sphere</type>
+              <radius>0.3</radius> -->
+              <type>fossen</type>
               <!-- Added mass: see p.28 in Berg2012 -->
-              <!-- <added_mass>
+              <added_mass>
                    779.79 -6.8773 -103.32  8.5426 -165.54 -7.8033
                   -6.8773    1222   51.29  409.44 -5.8488  62.726
@@ -25,13 +25,13 @@
                   -165.54 -5.8488 -386.42 -10.027  842.69 -1.1162
                   -7.8033  62.726  10.775  21.019 -1.1162  224.32
-              </added_mass> -->
+              </added_mass>
               <!-- Linear damping: see p.31 in Berg2012 -->
-              <!-- <linear_damping>
+              <linear_damping>
                   -74.82 -69.48 -728.4 -268.8 -309.77 -105
-              </linear_damping> -->
+              </linear_damping>
               <!-- Non-linear damping: see p.30 in Berg2012 -->
-              <!-- <quadratic_damping>
+              <quadratic_damping>
                   -748.22 -992.53 -1821.01 -672 -774.44 -523.27
-              </quadratic_damping> -->
+              </quadratic_damping>
             </hydrodynamic_model>
         </link>

File: ros_workspace/src/rov_description/urdf/rov_actuators.xacro (robot description, xacro)
@@ -13,21 +13,42 @@
     </xacro:thruster_module_first_order_basic_fcn_macro>
   </xacro:macro>
+  <!-- Thrusters rotate along the x-axis -->
+  <!-- The sign of the X-axis is in the opposite direction of the thrust -->
   <xacro:thruster_macro namespace="${namespace}" thruster_id="1">
-    <origin xyz="-0.1587 0.228 -0.14" rpy="${90*d2r} ${0*d2r} ${-225*d2r}"/>
+    <origin xyz="-0.1587 0.228 -0.14" rpy="${0*d2r} ${0*d2r} ${45*d2r}"/>
   </xacro:thruster_macro>
   <xacro:thruster_macro namespace="${namespace}" thruster_id="2">
-    <origin xyz="0.1587 0.228 -0.14" rpy="${90*d2r} ${0*d2r} ${225*d2r}"/>
+    <origin xyz="0.1587 0.228 -0.14" rpy="${0*d2r} ${0*d2r} ${135*d2r}"/>
   </xacro:thruster_macro>
   <xacro:thruster_macro namespace="${namespace}" thruster_id="3">
-    <origin xyz="0.16 -0.157 -0.132" rpy="${90*d2r} ${0*d2r} ${-45*d2r}"/>
+    <origin xyz="0.16 -0.157 -0.132" rpy="${0*d2r} ${0*d2r} ${-135*d2r}"/>
   </xacro:thruster_macro>
   <xacro:thruster_macro namespace="${namespace}" thruster_id="4">
-    <origin xyz="-0.16 -0.157 -0.132" rpy="${90*d2r} ${0*d2r} ${45*d2r}"/>
+    <origin xyz="-0.16 -0.157 -0.132" rpy="${0*d2r} ${0*d2r} ${-45*d2r}"/>
   </xacro:thruster_macro>
   <xacro:thruster_macro namespace="${namespace}" thruster_id="5">
-    <origin xyz="-0.25550 0.03394 -0.08263" rpy="${0*d2r} ${0*d2r} ${0*d2r}"/>
+    <origin xyz="-0.25550 0.03394 -0.08263" rpy="${0*d2r} ${90*d2r} ${0*d2r}"/>
   </xacro:thruster_macro>
   <xacro:thruster_macro namespace="${namespace}" thruster_id="6">
-    <origin xyz="0.25550 0.03394 -0.08263" rpy="${0*d2r} ${0*d2r} ${0*d2r}"/>
+    <origin xyz="0.25550 0.03394 -0.08263" rpy="${0*d2r} ${90*d2r} ${0*d2r}"/>
   </xacro:thruster_macro>
+  <!-- Color thruster propellers-->
+  <gazebo reference="${namespace}/thruster_1">
+    <material>Gazebo/Turquoise</material>
+  </gazebo>
+  <gazebo reference="${namespace}/thruster_2">
+    <material>Gazebo/Turquoise</material>
+  </gazebo>
+  <gazebo reference="${namespace}/thruster_3">
+    <material>Gazebo/Turquoise</material>
+  </gazebo>
+  <gazebo reference="${namespace}/thruster_4">
+    <material>Gazebo/Turquoise</material>
+  </gazebo>
+  <gazebo reference="${namespace}/thruster_5">
+    <material>Gazebo/Turquoise</material>
+  </gazebo>
+  <gazebo reference="${namespace}/thruster_6">
+    <material>Gazebo/Turquoise</material>
+  </gazebo>
 </robot>

File: ros_workspace/src/rov_description/urdf/rov_base.xacro (robot description, xacro)
@@ -19,8 +19,8 @@
       <inertial>
         <mass value="${mass}"/>
-        <origin xyz="0.0 0.0 -0.12001042"/> <!-- center of mass -->
-        <inertia ixx = "0.24968270"  ixy = "0.00003120"  ixz = "-0.00076418"
-                 iyx = "0.00003120"  iyy = "0.19606323"  iyz = "-0.01991623"
-                 izx = "-0.00076418" izy = "-0.01991623" izz = "0.22666109" />
+        <origin xyz="0.0 0.0 -0.12"/> <!-- center of mass -->
+        <inertia ixx = "0.24968270"  ixy = "0.0"  ixz = "0.0"
+                 iyx = "0.0"  iyy = "0.19606323"  iyz = "0.0"
+                 izx = "0.0" izy = "0.0" izz = "0.22666109" />
       </inertial>
       <visual>
@@ -63,4 +63,7 @@
       </collision>
     </link>
+    <gazebo reference="${namespace}/base_link">
+      <material>Gazebo/DarkGrey</material>
+    </gazebo>
     <!-- Set up hydrodynamic plugin given as input parameter -->
     <xacro:insert_block name="gazebo"/>
