Commit message: Switched sign on rotor constant and scaled the hydrodynamics for the ROV by a factor of 0.006

File: ros_workspace/src/rov_description/urdf/rov.gazebo.xacro (robot description, xacro)
@@ -1,5 +1,5 @@
 <?xml version="1.0"?>
 <robot xmlns:xacro="http://www.ros.org/wiki/xacro">
-    <xacro:property name="cob" value="0.0 0.0 0.01"/>
+    <xacro:property name="cob" value="0.00037196 0.001 0.01"/>
     <xacro:property name="volume" value="0.01"/>
     <xacro:macro name="rov_hydro_model" params="namespace">
@@ -18,19 +18,20 @@
               <type>fossen</type>
               <!-- Added mass: see p.28 in Berg2012 -->
+              <!-- RexROV hydrodynamics with a scale factor of 0.006 -->
               <added_mass>
-                   779.79 -6.8773 -103.32  8.5426 -165.54 -7.8033
-                  -6.8773    1222   51.29  409.44 -5.8488  62.726
-                  -103.32   51.29  3659.9  6.1112 -386.42  10.774
-                   8.5426  409.44  6.1112   534.9 -10.027  21.019
-                  -165.54 -5.8488 -386.42 -10.027  842.69 -1.1162
-                  -7.8033  62.726  10.775  21.019 -1.1162  224.32
+                   4.68      -0.041262  -0.61992  0.0512556   -0.99324 -0.0468198
+                  -0.0412638     7.332   0.30774    2.45664 -0.0350928   0.376356
+                  -0.61992     0.30756   21.9594  0.0366672   -2.31852   0.064644
+                   0.0512556   2.45664  0.036672     3.2094  -0.060162   0.126114
+                  -0.99324  -0.0350928  -2.31852  -0.060162    5.05614 -0.0066972
+                  -0.0468198  0.376356   0.06465   0.126114  -0.0066972   1.34592
               </added_mass>
               <!-- Linear damping: see p.31 in Berg2012 -->
               <linear_damping>
-                  -74.82 -69.48 -728.4 -268.8 -309.77 -105
+                  -0.44892 -0.41688 -4.3704 -1.6128 -1.85862 -0.63
               </linear_damping>
               <!-- Non-linear damping: see p.30 in Berg2012 -->
               <quadratic_damping>
-                  -748.22 -992.53 -1821.01 -672 -774.44 -523.27
+                  -4.48932 -5.95518 -10.92606 -4.032 4.64664 -3.13962
               </quadratic_damping>
             </hydrodynamic_model>

File: ros_workspace/src/rov_description/urdf/rov_actuators.xacro (robot description, xacro)
@@ -9,5 +9,5 @@
       mesh_filename="${prop_mesh_file}"
       dyn_time_constant="0.05"
-      rotor_constant="0.00031">
+      rotor_constant="-0.00031"> <!-- Negative rotor constant so that thrusters spin in the right direction -->
       <xacro:insert_block name="origin"/>
     </xacro:thruster_module_first_order_basic_fcn_macro>
@@ -16,20 +16,20 @@
   <!-- The sign of the X-axis is in the opposite direction of the thrust -->
   <xacro:thruster_macro namespace="${namespace}" thruster_id="1">
-    <origin xyz="-0.1587 0.228 -0.14" rpy="${0*d2r} ${0*d2r} ${45*d2r}"/>
+    <origin xyz="-0.15567119 0.23367751 -0.136" rpy="${0*d2r} ${0*d2r} ${45*d2r}"/>
   </xacro:thruster_macro>
   <xacro:thruster_macro namespace="${namespace}" thruster_id="2">
-    <origin xyz="0.1587 0.228 -0.14" rpy="${0*d2r} ${0*d2r} ${135*d2r}"/>
+    <origin xyz="0.15501313 0.23361171 -0.136" rpy="${0*d2r} ${0*d2r} ${135*d2r}"/>
   </xacro:thruster_macro>
   <xacro:thruster_macro namespace="${namespace}" thruster_id="3">
-    <origin xyz="0.16 -0.157 -0.132" rpy="${0*d2r} ${0*d2r} ${-135*d2r}"/>
+    <origin xyz="0.15497139 -0.15960511 -0.136" rpy="${0*d2r} ${0*d2r} ${-135*d2r}"/>
   </xacro:thruster_macro>
   <xacro:thruster_macro namespace="${namespace}" thruster_id="4">
-    <origin xyz="-0.16 -0.157 -0.132" rpy="${0*d2r} ${0*d2r} ${-45*d2r}"/>
+    <origin xyz="-0.15570687 -0.15963745 -0.136" rpy="${0*d2r} ${0*d2r} ${-45*d2r}"/>
   </xacro:thruster_macro>
   <xacro:thruster_macro namespace="${namespace}" thruster_id="5">
-    <origin xyz="-0.25550 0.03394 -0.08263" rpy="${0*d2r} ${90*d2r} ${0*d2r}"/>
+    <origin xyz="-0.25550103 0.03425058 -0.08012365" rpy="${0*d2r} ${90*d2r} ${0*d2r}"/>
   </xacro:thruster_macro>
   <xacro:thruster_macro namespace="${namespace}" thruster_id="6">
-    <origin xyz="0.25550 0.03394 -0.08263" rpy="${0*d2r} ${90*d2r} ${0*d2r}"/>
+    <origin xyz="0.25550103 0.03425058 -0.08012365" rpy="${0*d2r} ${90*d2r} ${0*d2r}"/>
   </xacro:thruster_macro>
   <!-- Color thruster propellers-->

File: ros_workspace/src/rov_description/urdf/rov_base.xacro (robot description, xacro)
@@ -19,5 +19,5 @@
       <inertial>
         <mass value="${mass}"/>
-        <origin xyz="0.0 0.0 -0.12"/> <!-- center of mass -->
+        <origin xyz="0.00056715 0.0005 -0.12"/> <!-- center of mass -->
         <inertia ixx = "0.24968270"  ixy = "0.0"  ixz = "0.0"
                  iyx = "0.0"  iyy = "0.19606323"  iyz = "0.0"

Commit message: Updated hydrodynamics and made a more functional model, the visual is not as good: thrusers dont line up with mesh

File: ros_workspace/src/rov_description/urdf/rov.gazebo.xacro (robot description, xacro)
@@ -2,5 +2,6 @@
 <robot xmlns:xacro="http://www.ros.org/wiki/xacro">
     <xacro:property name="cob" value="0.00037196 0.001 0.01"/>
-    <xacro:property name="volume" value="0.01"/>
+    <!-- ROV mass = 9.80543312 -->
+    <xacro:property name="volume" value="0.0099"/> <!-- ROV is slightly positively bouyant at 0.0099m^3 -->
     <xacro:macro name="rov_hydro_model" params="namespace">
         <link name="${namespace}/base_link">
@@ -18,5 +19,5 @@
               <type>fossen</type>
               <!-- Added mass: see p.28 in Berg2012 -->
-              <!-- RexROV hydrodynamics with a scale factor of 0.006 -->
+              <!-- RexROV hydrodynamics with a scale factor of 0.006 - rough estimate but seems to work well-->
               <added_mass>
                    4.68      -0.041262  -0.61992  0.0512556   -0.99324 -0.0468198

File: ros_workspace/src/rov_description/urdf/rov_actuators.xacro (robot description, xacro)
@@ -14,16 +14,16 @@
   </xacro:macro>
   <!-- Thrusters rotate along the x-axis -->
-  <!-- The sign of the X-axis is in the opposite direction of the thrust -->
+  <!-- The sign of the X-axis is in the opposite direction as the thrust -->
   <xacro:thruster_macro namespace="${namespace}" thruster_id="1">
-    <origin xyz="-0.15567119 0.23367751 -0.136" rpy="${0*d2r} ${0*d2r} ${45*d2r}"/>
+    <origin xyz="-0.15567119 0.23361171 -0.136" rpy="${0*d2r} ${0*d2r} ${45*d2r}"/>
   </xacro:thruster_macro>
   <xacro:thruster_macro namespace="${namespace}" thruster_id="2">
-    <origin xyz="0.15501313 0.23361171 -0.136" rpy="${0*d2r} ${0*d2r} ${135*d2r}"/>
+    <origin xyz="0.15567119 0.23361171 -0.136" rpy="${0*d2r} ${0*d2r} ${135*d2r}"/>
   </xacro:thruster_macro>
   <xacro:thruster_macro namespace="${namespace}" thruster_id="3">
-    <origin xyz="0.15497139 -0.15960511 -0.136" rpy="${0*d2r} ${0*d2r} ${-135*d2r}"/>
+    <origin xyz="0.15497139 -0.15963745 -0.136" rpy="${0*d2r} ${0*d2r} ${-135*d2r}"/>
   </xacro:thruster_macro>
   <xacro:thruster_macro namespace="${namespace}" thruster_id="4">
-    <origin xyz="-0.15570687 -0.15963745 -0.136" rpy="${0*d2r} ${0*d2r} ${-45*d2r}"/>
+    <origin xyz="-0.15497139 -0.15963745 -0.136" rpy="${0*d2r} ${0*d2r} ${-45*d2r}"/>
   </xacro:thruster_macro>
   <xacro:thruster_macro namespace="${namespace}" thruster_id="5">

File: ros_workspace/src/rov_description/urdf/rov_default.xacro (robot description, xacro)
@@ -25,5 +25,5 @@
   <!-- setup base links -->
   <link name="${namespace}/frame_link"/>
-  <joint name="${namespace}/base_link_joint" type="fixed">
+  <joint name="${namespace}/base_frame_joint" type="fixed">
     <parent link="${namespace}/base_link"/>
     <child link="${namespace}/frame_link"/>

Commit message: Removed thruster noise temporarily and changed quadratic dampening hydrodynamics to work better in the simulation

File: ros_workspace/src/rov_description/urdf/rov.gazebo.xacro (robot description, xacro)
@@ -3,5 +3,5 @@
     <xacro:property name="cob" value="0.00037196 0.001 0.01"/>
     <!-- ROV mass = 9.80543312 -->
-    <xacro:property name="volume" value="0.0099"/> <!-- ROV is slightly positively bouyant at 0.0099m^3 -->
+    <xacro:property name="volume" value="0.00985"/> <!-- ROV is slightly positively bouyant at 0.0099m^3 -->
     <xacro:macro name="rov_hydro_model" params="namespace">
         <link name="${namespace}/base_link">
@@ -33,6 +33,9 @@
               </linear_damping>
               <!-- Non-linear damping: see p.30 in Berg2012 -->
+              <!-- <quadratic_damping>
+                  -4.48932 -5.95518 -10.92606 -4.032 -4.64664 -3.13962
+              </quadratic_damping> -->
               <quadratic_damping>
-                  -4.48932 -5.95518 -10.92606 -4.032 4.64664 -3.13962
+                  -6 -8 -12 -25 -25 -5
               </quadratic_damping>
             </hydrodynamic_model>

File: ros_workspace/src/rov_description/urdf/rov_actuators.xacro (robot description, xacro)
@@ -15,15 +15,16 @@
   <!-- Thrusters rotate along the x-axis -->
   <!-- The sign of the X-axis is in the opposite direction as the thrust -->
+  <!-- If necessary to put all thrusters on same z-plane then use the value -0.36 -->
   <xacro:thruster_macro namespace="${namespace}" thruster_id="1">
-    <origin xyz="-0.15567119 0.23361171 -0.136" rpy="${0*d2r} ${0*d2r} ${45*d2r}"/>
+    <origin xyz="-0.15567119 0.23361171 -0.14" rpy="${0*d2r} ${0*d2r} ${45*d2r}"/>
   </xacro:thruster_macro>
   <xacro:thruster_macro namespace="${namespace}" thruster_id="2">
-    <origin xyz="0.15567119 0.23361171 -0.136" rpy="${0*d2r} ${0*d2r} ${135*d2r}"/>
+    <origin xyz="0.15567119 0.23361171 -0.14" rpy="${0*d2r} ${0*d2r} ${135*d2r}"/>
   </xacro:thruster_macro>
   <xacro:thruster_macro namespace="${namespace}" thruster_id="3">
-    <origin xyz="0.15567119 -0.15963745 -0.136" rpy="${0*d2r} ${0*d2r} ${-135*d2r}"/>
+    <origin xyz="0.15567119 -0.15963745 -0.132" rpy="${0*d2r} ${0*d2r} ${-135*d2r}"/>
   </xacro:thruster_macro>
   <xacro:thruster_macro namespace="${namespace}" thruster_id="4">
-    <origin xyz="-0.15567119 -0.15963745 -0.136" rpy="${0*d2r} ${0*d2r} ${-45*d2r}"/>
+    <origin xyz="-0.15567119 -0.15963745 -0.132" rpy="${0*d2r} ${0*d2r} ${-45*d2r}"/>
   </xacro:thruster_macro>
   <xacro:thruster_macro namespace="${namespace}" thruster_id="5">
